File: Audio.kicad_sch (KiCad schematic)
At the start: 25 parts, among them J5 JST PH2.0-1x2, J6 JST PH2.0-1x2, U10 MEMS Microphone, U7 ES7149, U8 NS4150, U9 NS4150

Commit message: release evt2
Signed-off-by: Sean Cross <sean@xobs.io>
Parts:
- R12, R13, R14, R21: value R 20k 0201 -> R 22.1k 0201; symbol Galvani:R 20k 0201 -> Galvani:R 22.1k 0201; Val 20k -> 22.1k
Changed lines of the file:
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@@
 	)
 	(symbol
-		(lib_id "Galvani:R 20k 0201")
+		(lib_id "Galvani:R 22.1k 0201")
 		(at 167.64 101.6 270)
 		(unit 1)
@@
 			)
 		)
-		(property "Value" "R 20k 0201"
+		(property "Value" "R 22.1k 0201"
 			(at 167.64 110.49 90)
 			(effects
@@
 			)
 		)
-		(property "Val" "20k"
+		(property "Val" "22.1k"
 			(at 167.64 102.87 90)
 			(effects
@@
 	)
 	(symbol
-		(lib_id "Galvani:R 20k 0201")
+		(lib_id "Galvani:R 22.1k 0201")
 		(at 166.37 66.04 270)
 		(unit 1)
@@
 			)
 		)
-		(property "Value" "R 20k 0201"
+		(property "Value" "R 22.1k 0201"
 			(at 166.37 74.93 90)
 			(effects
@@
 			)
 		)
-		(property "Val" "20k"
+		(property "Val" "22.1k"
 			(at 169.418 65.024 90)
 			(effects
@@
 	)
 	(symbol
-		(lib_id "Galvani:R 20k 0201")
+		(lib_id "Galvani:R 22.1k 0201")
 		(at 167.64 99.06 270)
 		(unit 1)
@@
 			)
 		)
-		(property "Value" "R 20k 0201"
+		(property "Value" "R 22.1k 0201"
 			(at 167.64 107.95 90)
 			(effects
@@
 			)
 		)
-		(property "Val" "20k"
+		(property "Val" "22.1k"
 			(at 167.64 100.33 90)
 			(effects
@@
 	)
 	(symbol
-		(lib_id "Galvani:R 20k 0201")
+		(lib_id "Galvani:R 22.1k 0201")
 		(at 166.37 63.5 270)
 		(unit 1)
@@
 			)
 		)
-		(property "Value" "R 20k 0201"
+		(property "Value" "R 22.1k 0201"
 			(at 166.37 72.39 90)
 			(effects
@@
 			)
 		)
-		(property "Val" "20k"
+		(property "Val" "22.1k"
 			(at 169.418 62.484 90)
 			(effects
