File: CPU.kicad_sch (KiCad schematic)
At the start: 34 parts, among them J1 USB-C Receptacle, J2 U.FL Connector, P1 Cap 2.4pF 0201, P2 L 2.7nH 0201, P3 Cap 3.9pF 0201, P7 L 2.7nH 0201, SW1 Pushbutton 4.2x3.2mm 250gf, SW2 Pushbutton 4.2x3.2mm 250gf, U2 ESP32-S3, U3 W25Q128JVS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

Commit message: release evt2
Signed-off-by: Sean Cross <sean@xobs.io>
Parts:
- C10, C50, C51, C52, C53, C9: LCSC C307380 -> (none); MPN CL03A104KO3NNNC -> (none); Manufacturer Samsung Electro-Mechanics -> (none)
- C49: LCSC C76935 -> (none); MPN GRM033R61A105ME44D -> (none); Manufacturer Murata Electronics -> (none)
- P2, P7: LCSC C206439 -> C237548; MPN LQP03TN2N2C02D -> LQP03PN2N7C02D
- R5, R6, R7, R8, R9: value R 20k 0201 -> R 22.1k 0201; symbol Galvani:R 20k 0201 -> Galvani:R 22.1k 0201; Val 20k -> 22.1k
Connections:
- net I2S_BCLK: now also U2.45 (MTDO/JTAG/GPIO40); no longer U2.50 (U0RXD/PROG/GPIO44)
- net I2S_IN: now also U2.44 (MTCK/JTAG/GPIO39); no longer U2.48 (MTMS/JTAG/GPIO42)
- net I2S_LRCK: now also U2.43 (GPIO38); no longer U2.44 (MTCK/JTAG/GPIO39)
- net I2S_MCLK: now also U2.15 (GPIO10/ADC1_CH9); no longer U2.45 (MTDO/JTAG/GPIO40)
- net I2S_OUT: now also U2.14 (GPIO9/ADC1_CH8); no longer U2.47 (MTDI/JTAG/GPIO41)
