File: Heirarchy.kicad_sch (KiCad schematic)
At the start: 3 parts

Commit message: release evt2
Signed-off-by: Sean Cross <sean@xobs.io>
Connections:
- net GND: now also TP1.1; no longer TP2.1
- net V5V: now also TP2.1; no longer TP1.1
Other:
- moved on the sheet: TP1, TP2
Changed lines of the file:
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@@
 	(generator_version "8.0")
 	(paper "A4")
+	(title_block
+		(date "2024-10-09")
+		(rev "EVT2")
+	)
 	(bus
 		(pts
-			(xy 96.52 139.7) (xy 128.27 139.7)
+			(xy 115.57 91.44) (xy 147.32 91.44)
 		)
 		(stroke
@@
 	(bus
 		(pts
-			(xy 96.52 154.94) (xy 128.27 154.94)
+			(xy 115.57 110.49) (xy 147.32 110.49)
 		)
 		(stroke
@@
 	(wire
 		(pts
-			(xy 96.52 142.24) (xy 128.27 142.24)
+			(xy 115.57 93.98) (xy 147.32 93.98)
 		)
 		(stroke
@@
 	(wire
 		(pts
-			(xy 96.52 129.54) (xy 128.27 129.54)
+			(xy 115.57 76.2) (xy 147.32 76.2)
 		)
 		(stroke
@@
 	(wire
 		(pts
-			(xy 96.52 127) (xy 128.27 127)
+			(xy 115.57 73.66) (xy 147.32 73.66)
 		)
 		(stroke
@@
 	)
 	(rectangle
-		(start 137.16 91.44)
-		(end 207.01 107.95)
+		(start 92.71 135.89)
+		(end 162.56 152.4)
 		(stroke
 			(width 0)
@@
 	(text "Test Points and Mounting Holes"
 		(exclude_from_sim no)
-		(at 138.938 107.188 0)
+		(at 94.488 151.638 0)
 		(effects
 			(font
@@
 	(symbol
 		(lib_id "Galvani:V5V")
-		(at 182.88 97.79 0)
+		(at 149.86 142.24 0)
 		(unit 1)
 		(exclude_from_sim no)
@@
 		(dnp no)
 		(property "Reference" "#PWR063"
-			(at 182.88 101.6 0)
+			(at 149.86 146.05 0)
 			(effects
 				(font
@@
 		)
 		(property "Value" "V5V"
-			(at 182.88 95.504 0)
+			(at 149.86 139.954 0)
 			(effects
 				(font
@@
 		)
 		(property "Footprint" ""
-			(at 182.88 97.79 0)
+			(at 149.86 142.24 0)
 			(effects
 				(font
@@
 		)
 		(property "Datasheet" ""
-			(at 182.88 97.79 0)
+			(at 149.86 142.24 0)
 			(effects
 				(font
@@
 		)
 		(property "Description" ""
-			(at 182.88 97.79 0)
+			(at 149.86 142.24 0)
 			(effects
 				(font
@@
 	(symbol
 		(lib_id "Connector:TestPoint")
-		(at 194.31 97.79 270)
+		(at 149.86 142.24 270)
 		(unit 1)
 		(exclude_from_sim no)
@@
 		(fields_autoplaced yes)
 		(property "Reference" "TP2"
-			(at 199.39 96.5199 90)
+			(at 154.94 140.9699 90)
 			(effects
 				(font
@@
 		)
 		(property "Value" "GND"
-			(at 199.39 99.0599 90)
+			(at 154.94 143.5099 90)
 			(effects
 				(font
@@
 		)
 		(property "Footprint" "Galvani:Test Point"
-			(at 194.31 102.87 0)
+			(at 149.86 147.32 0)
 			(effects
 				(font
@@
 		)
 		(property "Datasheet" "~"
-			(at 194.31 102.87 0)
+			(at 149.86 147.32 0)
 			(effects
 				(font
@@
 		)
 		(property "Description" "test point"
-			(at 194.31 97.79 0)
+			(at 149.86 142.24 0)
 			(effects
 				(font
@@
 	(symbol
 		(lib_id "Connector:TestPoint")
-		(at 182.88 97.79 270)
+		(at 138.43 142.24 270)
 		(unit 1)
 		(exclude_from_sim no)
@@
 		(fields_autoplaced yes)
 		(property "Reference" "TP1"
-			(at 187.96 96.5199 90)
+			(at 143.51 140.9699 90)
 			(effects
 				(font
@@
 		)
 		(property "Value" "5V"
-			(at 187.96 99.0599 90)
+			(at 143.51 143.5099 90)
 			(effects
 				(font
@@
 		)
 		(property "Footprint" "Galvani:Test Point"
-			(at 182.88 102.87 0)
+			(at 138.43 147.32 0)
 			(effects
 				(font
@@
 		)
 		(property "Datasheet" "~"
-			(at 182.88 102.87 0)
+			(at 138.43 147.32 0)
 			(effects
 				(font
@@
 		)
 		(property "Description" "test point"
-			(at 182.88 97.79 0)
+			(at 138.43 142.24 0)
 			(effects
 				(font
@@
 	(symbol
 		(lib_id "power:GND")
-		(at 194.31 97.79 0)
+		(at 138.43 142.24 0)
 		(unit 1)
 		(exclude_from_sim no)
@@
 		(fields_autoplaced yes)
 		(property "Reference" "#PWR084"
-			(at 194.31 104.14 0)
+			(at 138.43 148.59 0)
 			(effects
 				(font
@@
 		)
 		(property "Value" "GND"
-			(at 194.31 102.87 0)
+			(at 138.43 147.32 0)
 			(effects
 				(font
@@
 		)
 		(property "Footprint" ""
-			(at 194.31 97.79 0)
+			(at 138.43 142.24 0)
 			(effects
 				(font
@@
 		)
 		(property "Datasheet" ""
-			(at 194.31 97.79 0)
+			(at 138.43 142.24 0)
 			(effects
 				(font
@@
 		)
 		(property "Description" ""
-			(at 194.31 97.79 0)
+			(at 138.43 142.24 0)
 			(effects
 				(font
@@
 	(symbol
 		(lib_id "Mechanical:MountingHole")
-		(at 142.24 97.79 0)
+		(at 97.79 142.24 0)
 		(unit 1)
 		(exclude_from_sim yes)
@@
 		(dnp no)
 		(property "Reference" "H2"
-			(at 144.78 96.5199 0)
+			(at 100.33 140.9699 0)
 			(effects
 				(font
@@
 		)
 		(property "Value" "Mounting Hole"
-			(at 144.78 97.79 0)
+			(at 100.33 142.24 0)
 			(effects
 				(font
@@
 		)
 		(property "Footprint" "MountingHole:MountingHole_3.5mm"
-			(at 142.24 97.79 0)
+			(at 97.79 142.24 0)
 			(effects
 				(font
@@
 		)
 		(property "Datasheet" "~"
-			(at 142.24 97.79 0)
+			(at 97.79 142.24 0)
 			(effects
 				(font
@@
 		)
 		(property "Description" "Mounting Hole without connection"
-			(at 142.24 97.79 0)
+			(at 97.79 142.24 0)
 			(effects
 				(font
@@
 	)
 	(sheet
-		(at 74.295 124.46)
-		(size 22.225 34.29)
+		(at 93.345 71.12)
+		(size 22.225 46.99)
 		(fields_autoplaced yes)
 		(stroke
@@
 		)
 		(property "Sheetname" "CPU"
-			(at 74.295 123.7484 0)
-			(effects
-				(font
-					(size 1.27 1.27)
+			(at 93.345 69.1384 0)
+			(effects
+				(font
+					(size 3.81 3.81)
 				)
 				(justify left bottom)
@@
 		)
 		(property "Sheetfile" "CPU.kicad_sch"
-			(at 74.295 159.3346 0)
+			(at 93.345 118.6946 0)
 			(effects
 				(font
@@
 		)
 		(pin "LED_EXTERNAL" output
-			(at 96.52 127 0)
+			(at 115.57 73.66 0)
 			(effects
 				(font
@@
 		)
 		(pin "{I2S}" output
-			(at 96.52 139.7 0)
+			(at 115.57 91.44 0)
 			(effects
 				(font
@@
 		)
 		(pin "LED_INTERNAL" output
-			(at 96.52 129.54 0)
+			(at 115.57 76.2 0)
 			(effects
 				(font
@@
 		)
 		(pin "AUDIO_EN" output
-			(at 96.52 142.24 0)
+			(at 115.57 93.98 0)
 			(effects
 				(font
@@
 		)
 		(pin "{SD}" bidirectional
-			(at 96.52 154.94 0)
+			(at 115.57 110.49 0)
 			(effects
 				(font
@@
 	)
 	(sheet
-		(at 128.27 152.4)
+		(at 147.32 107.95)
 		(size 15.24 10.16)
 		(fields_autoplaced yes)
@@
 		)
 		(property "Sheetname" "SD Card"
-			(at 128.27 151.6884 0)
-			(effects
-				(font
-					(size 1.27 1.27)
+			(at 147.32 105.9684 0)
+			(effects
+				(font
+					(size 3.81 3.81)
 				)
 				(justify left bottom)
@@
 		)
 		(property "Sheetfile" "SDCard.kicad_sch"
-			(at 128.27 163.1446 0)
+			(at 147.32 118.6946 0)
 			(effects
 				(font
@@
 		)
 		(pin "{SD}" bidirectional
-			(at 128.27 154.94 180)
+			(at 147.32 110.49 180)
 			(effects
 				(font
@@
 	)
 	(sheet
-		(at 128.27 138.43)
+		(at 147.32 90.17)
 		(size 16.51 7.62)
 		(fields_autoplaced yes)
@@
 		)
 		(property "Sheetname" "Audio"
-			(at 128.27 137.7184 0)
-			(effects
-				(font
-					(size 1.27 1.27)
+			(at 147.32 88.1884 0)
+			(effects
+				(font
+					(size 3.81 3.81)
 				)
 				(justify left bottom)
@@
 		)
 		(property "Sheetfile" "Audio.kicad_sch"
-			(at 128.27 146.6346 0)
+			(at 147.32 98.3746 0)
 			(effects
 				(font
@@
 		)
 		(pin "{I2S}" input
-			(at 128.27 139.7 180)
+			(at 147.32 91.44 180)
 			(effects
 				(font
@@
 		)
 		(pin "AUDIO_EN" input
-			(at 128.27 142.24 180)
+			(at 147.32 93.98 180)
 			(effects
 				(font
@@
 	)
 	(sheet
-		(at 128.27 124.46)
+		(at 147.32 71.12)
 		(size 22.86 8.89)
 		(fields_autoplaced yes)
@@
 		)
 		(property "Sheetname" "LEDs"
-			(at 128.27 123.7484 0)
-			(effects
-				(font
-					(size 1.27 1.27)
+			(at 147.32 69.1384 0)
+			(effects
+				(font
+					(size 3.81 3.81)
 				)
 				(justify left bottom)
@@
 		)
 		(property "Sheetfile" "LEDs.kicad_sch"
-			(at 128.27 133.9346 0)
+			(at 147.32 80.5946 0)
 			(effects
 				(font
@@
 		)
 		(pin "LED_INTERNAL" input
-			(at 128.27 129.54 180)
+			(at 147.32 76.2 180)
 			(effects
 				(font
@@
 		)
 		(pin "LED_EXTERNAL" input
-			(at 128.27 127 180)
+			(at 147.32 73.66 180)
 			(effects
 				(font
@@
 	)
 	(sheet
-		(at 75.565 98.425)
-		(size 30.48 7.62)
+		(at 94.615 45.085)
+		(size 55.245 6.985)
 		(fields_autoplaced yes)
 		(stroke
@@
 		)
 		(property "Sheetname" "Power"
-			(at 75.565 97.7134 0)
+			(at 94.615 44.3734 0)
 			(effects
 				(font
@@
 		)
 		(property "Sheetfile" "Power.kicad_sch"
-			(at 75.565 106.6296 0)
-			(effects
-				(font
+			(at 94.615 52.6546 0)
+			(effects
+				(font
