File: SDCard.kicad_sch (KiCad schematic)
At the start: 6 parts, among them J8 Micro SD Card

Commit message: release evt2
Signed-off-by: Sean Cross <sean@xobs.io>
Parts:
- R22, R23, R24, R25: value R 20k 0201 -> R 22.1k 0201; symbol Galvani:R 20k 0201 -> Galvani:R 22.1k 0201; Val 20k -> 22.1k
Changed lines of the file:
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@@
 	)
 	(symbol
-		(lib_id "Galvani:R 20k 0201")
+		(lib_id "Galvani:R 22.1k 0201")
 		(at 123.19 80.01 0)
 		(mirror x)
@@
 			)
 		)
-		(property "Value" "R 20k 0201"
+		(property "Value" "R 22.1k 0201"
 			(at 132.08 80.01 90)
 			(effects
@@
 			)
 		)
-		(property "Val" "20k"
+		(property "Val" "22.1k"
 			(at 124.46 80.01 90)
 			(effects
@@
 	)
 	(symbol
-		(lib_id "Galvani:R 20k 0201")
+		(lib_id "Galvani:R 22.1k 0201")
 		(at 128.27 80.01 0)
 		(mirror x)
@@
 			)
 		)
-		(property "Value" "R 20k 0201"
+		(property "Value" "R 22.1k 0201"
 			(at 137.16 80.01 90)
 			(effects
@@
 			)
 		)
-		(property "Val" "20k"
+		(property "Val" "22.1k"
 			(at 129.54 80.01 90)
 			(effects
@@
 	)
 	(symbol
-		(lib_id "Galvani:R 20k 0201")
+		(lib_id "Galvani:R 22.1k 0201")
 		(at 113.03 80.01 0)
 		(mirror x)
@@
 			)
 		)
-		(property "Value" "R 20k 0201"
+		(property "Value" "R 22.1k 0201"
 			(at 121.92 80.01 90)
 			(effects
@@
 			)
 		)
-		(property "Val" "20k"
+		(property "Val" "22.1k"
 			(at 114.3 80.01 90)
 			(effects
@@
 	)
 	(symbol
-		(lib_id "Galvani:R 20k 0201")
+		(lib_id "Galvani:R 22.1k 0201")
 		(at 118.11 80.01 0)
 		(mirror x)
@@
 			)
 		)
-		(property "Value" "R 20k 0201"
+		(property "Value" "R 22.1k 0201"
 			(at 127 80.01 90)
 			(effects
@@
 			)
 		)
-		(property "Val" "20k"
+		(property "Val" "22.1k"
 			(at 119.38 80.01 90)
 			(effects
